File: ProtoBoard_V1/MOSAIC ProtoBoard.kicad_sch (KiCad schematic)
At the start: 11 parts, among them J7 Qwiic Adapter, J8 Qwiic Adapter, J9 Qwiic Adapter

Commit message: Add mounting holes to schematic
Parts:
- added H10, H9: MountingHole_Pad, main_board_footprints_V1.0:MountingHole_3.2mm_Pad_Oval, symbol Mechanical:MountingHole_Pad
- added H7, H8: MountingHole_Pad, MountingHole:MountingHole_3.2mm_M3_Pad, symbol Mechanical:MountingHole_Pad
Connections:
- net GND: now also H10.1, H7.1, H8.1, H9.1

Commit message: Add mounts to schem and board
Parts:
- H10, H9: footprint main_board_footprints_V1.0:MountingHole_3.2mm_Pad_Oval -> protoboard_footprints_V1.0:MountingHole_3.2mm_Pad_Oval
Changed lines of the file:
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@@
 			)
 		)
-		(property "Footprint" "main_board_footprints_V1.0:MountingHole_3.2mm_Pad_Oval"
+		(property "Footprint" "protoboard_footprints_V1.0:MountingHole_3.2mm_Pad_Oval"
 			(at 25.4 177.8 0)
 			(effects
@@
 			)
 		)
-		(property "Footprint" "main_board_footprints_V1.0:MountingHole_3.2mm_Pad_Oval"
+		(property "Footprint" "protoboard_footprints_V1.0:MountingHole_3.2mm_Pad_Oval"
 			(at 25.4 189.23 0)
 			(effects
